File: acs-display-grabber.kicad_pcb (KiCad board)
At the start: 2 copper layers, 32 parts, among them IC1 ATMEGA328P-P, U1 74HC14, U2 74HC14

Commit message: version 2
Parts:
- removed BUTTONS1: CONN_01X05, Pin_Headers:Pin_Header_Angled_1x04
- removed CRYSTAL1: CRYSTAL, Crystals:Crystal_HC49-U_Vertical
- removed D5, D6, D7, D8, D9: ZF 3.9, Diodes_ThroughHole:Diode_DO-35_SOD27_Horizontal_RM10
- removed DISPLAY1: CONN_01x09, Pin_Headers:Pin_Header_Angled_1x09
- removed I2C_PORT1: CONN_01x04, Pin_Headers:Pin_Header_Angled_1x05
- removed IC1: ATMEGA328P-P, Housings_DIP:DIP-28_W7.62mm
- removed ISP_PORT1: CONN_02X03, Pin_Headers:Pin_Header_Angled_2x03
- removed SUMMER,1: CONN_01X04, Pin_Headers:Pin_Header_Angled_1x04
- removed U2: 74HC14, Housings_DIP:DIP-14_W7.62mm
- added C4: 10nF, Capacitors_SMD:C_0805, F.Cu at (155.0, 94.9)
- added C5: 10nF, Capacitors_SMD:C_0805, F.Cu at (153.7, 80.7)
- added C6: 20nF, Capacitors_SMD:C_0805, F.Cu at (187.2, 110.7)
- added C7: 10nF, Capacitors_SMD:C_0805, F.Cu at (152.4, 101.0)
- added C8: 10nF, Capacitors_SMD:C_0805, F.Cu at (151.1, 84.2)
- added C9: 20nF, Capacitors_SMD:C_0805, F.Cu at (187.2, 129.0)
- added G***: LOGO, acs-display-grabber:logo_front, B.Cu at (128.0, 119.0)
- added G***: LOGO, acs-display-grabber:logo2_front, F.Cu at (124.0, 115.0)
- added P1: CONN_02X07, Pin_Headers:Pin_Header_Angled_2x07, F.Cu at (117.5, 88.8)
- added P2: CONN_02X04, Pin_Headers:Pin_Header_Angled_2x04, F.Cu at (184.5, 66.6)
- added R12: 3.3K, Resistors_SMD:R_0805, F.Cu at (190.8, 108.6)
- added R13: 3.3K, Resistors_SMD:R_0805, F.Cu at (187.3, 125.9)
- added REF**: MountingHole_3mm, Mounting_Holes:MountingHole_3mm, F.Cu at (199.0, 132.0)
- added REF**: MountingHole_3mm, Mounting_Holes:MountingHole_3mm, F.Cu at (109.0, 132.0)
- added REF**: MountingHole_3mm, Mounting_Holes:MountingHole_3mm, F.Cu at (199.0, 58.0)
- added REF**: MountingHole_3mm, Mounting_Holes:MountingHole_3mm, F.Cu at (109.0, 58.0)
- added RV1: POT, ACP CA6:ACP_CA6, F.Cu at (135.7, 64.7)
- added RV2: POT, ACP CA6:ACP_CA6, F.Cu at (137.8, 110.2)
- added U3: LM393, Housings_SOIC:SOIC-8_3.9x4.9mm_Pitch1.27mm, F.Cu at (135.7, 101.5)
- added U4: LM339, Housings_SOIC:SOIC-14_3.9x8.7mm_Pitch1.27mm, F.Cu at (135.7, 76.1)
- added U5: 74LS573, Housings_SOIC:SOIC-20_7.5x12.8mm_Pitch1.27mm, F.Cu at (166.1, 73.6)
- added U6: 74LS573, Housings_SOIC:SOIC-20_7.5x12.8mm_Pitch1.27mm, F.Cu at (166.1, 90.1)
- added U7: 74LS573, Housings_SOIC:SOIC-20_7.5x12.8mm_Pitch1.27mm, F.Cu at (166.1, 106.6)
- added U8: 74LS573, Housings_SOIC:SOIC-20_7.5x12.8mm_Pitch1.27mm, F.Cu at (166.1, 123.1)
- added U9: MCP23017, Housings_SOIC:SOIC-28_7.5x17.9mm_Pitch1.27mm, F.Cu at (187.7, 81.2)
- C1: value 22pF -> 20nF; footprint Capacitors_ThroughHole:C_Rect_L7_W2.5_P5 -> Capacitors_SMD:C_0805
- C2: value 22pF -> 10nF; footprint Capacitors_ThroughHole:C_Rect_L7_W2.5_P5 -> Capacitors_SMD:C_0805
- C3: value 100uF -> 20nF; footprint Capacitors_Elko_ThroughHole:Elko_vert_11.2x6.3mm_RM2.5 -> Capacitors_SMD:C_0805
- D1, D2, D3, D4: value ZF 3.9 -> 1N4007; footprint Diodes_ThroughHole:Diode_DO-35_SOD27_Horizontal_RM10 -> Diodes_SMD:MELF_Handsoldering
- R1, R2, R3, R4: value 470k -> 1.8K; footprint Resistors_ThroughHole:Resistor_Horizontal_RM10mm -> Resistors_SMD:R_0805
- R10, R11, R5, R6, R7, R8, R9: value 470k -> 3.3K; footprint Resistors_ThroughHole:Resistor_Horizontal_RM10mm -> Resistors_SMD:R_0805
- U1: value 74HC14 -> LM339; footprint Housings_DIP:DIP-14_W7.62mm -> Housings_SOIC:SOIC-14_3.9x8.7mm_Pitch1.27mm
- moved R1 169.3 mm to (201.4, 76.1)
- moved R4 149.9 mm to (178.6, 125.4), turned to 0 degrees
- moved R3 149.5 mm to (179.1, 114.7), turned to 0 degrees
- moved R2 147.9 mm to (178.6, 100.5), turned to 0 degrees
- moved D4 135.8 mm to (178.6, 129.0)
- moved D3 123.1 mm to (179.1, 110.7)
- moved D1 121.0 mm to (197.4, 68.5), turned to 90 degrees
- moved R5 120.1 mm to (145.0, 129.5), turned to 0 degrees
- moved R6 115.2 mm to (145.0, 126.5), turned to 0 degrees
- moved D2 113.8 mm to (178.6, 96.4)
- moved R11 110.7 mm to (179.1, 92.9), turned to 180 degrees
- moved R7 110.4 mm to (145.0, 123.4), turned to 0 degrees
- moved R8 105.5 mm to (145.0, 120.4), turned to 0 degrees
- moved R9 100.6 mm to (145.0, 117.3), turned to 0 degrees
- moved C1 84.6 mm to (197.4, 78.2), turned to 270 degrees
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Connections:
- net Net-(D3-Pad2) renamed /COM2clean
- net Net-(D4-Pad2) renamed /COM3clean
- C1 pad 2: Earth -> +5V
- C2 pad 1: Net-(C2-Pad1) -> +5V
- C2 pad 2: Earth -> /SEG0clean
- C3 pad 1: VCC -> Net-(C3-Pad1)
- C3 pad 2: Earth -> +5V
- D1 pad 1: Net-(D1-Pad1) -> Net-(C1-Pad1)
- D1 pad 2: Net-(D1-Pad2) -> /COM0clean
- D2 pad 1: Net-(D2-Pad1) -> Net-(C3-Pad1)
- D2 pad 2: Net-(D2-Pad2) -> /COM1clean
- D3 pad 1: Net-(D3-Pad1) -> Net-(C6-Pad1)
- D4 pad 1: Net-(D4-Pad1) -> Net-(C9-Pad1)
- R1 pad 1: Net-(D1-Pad2) -> /COM0clean
- R1 pad 2: Earth -> Net-(C1-Pad1)
- R10 pad 1: Earth -> +5V
- R10 pad 2: Net-(BUTTONS1-Pad3) -> /COM0clean
- R11 pad 1: Earth -> +5V
- R11 pad 2: Net-(BUTTONS1-Pad2) -> /COM1clean
- R2 pad 1: Net-(D2-Pad2) -> /COM1clean
- R2 pad 2: Earth -> Net-(C3-Pad1)
- R3 pad 2: Earth -> Net-(C6-Pad1)
- R4 pad 2: Earth -> Net-(C9-Pad1)
- R5 pad 1: Net-(D5-Pad2) -> +5V
- R5 pad 2: Earth -> /SEG0clean
- R6 pad 1: Net-(D6-Pad2) -> +5V
- R6 pad 2: Earth -> /SEG1clean
- R7 pad 1: Net-(D7-Pad2) -> +5V
- R7 pad 2: Earth -> /SEG2clean
- R8 pad 1: Net-(D8-Pad2) -> +5V
- R8 pad 2: Earth -> /SEG3clean
- R9 pad 1: Net-(D9-Pad2) -> +5V
- R9 pad 2: Earth -> /SEG4clean
- U1 pad 1: Net-(D1-Pad1) -> /SEG1clean
- U1 pad 10: /DISP6 -> /SEG2
- U1 pad 11: Net-(D6-Pad1) -> /Vlow
- U1 pad 12: /DISP5 -> GND
- U1 pad 13: Net-(D5-Pad1) -> /SEG2clean
- U1 pad 14: VCC -> /SEG3clean
- U1 pad 2: /DISP1 -> /SEG0clean
- U1 pad 3: Net-(D2-Pad1) -> +5V
- U1 pad 4: /DISP2 -> /SEG0
- U1 pad 5: Net-(D3-Pad1) -> /Vlow
- U1 pad 6: /DISP3 -> /SEG1
- U1 pad 7: Earth -> /Vlow
- U1 pad 8: /DISP4 -> /SEG3
- U1 pad 9: Net-(D4-Pad1) -> /Vlow
Routing:
- net +5V: track 0.00 -> 432.8 mm, vias 0 -> 12
- net Earth: track 289.2 -> 0.00 mm, vias 4 -> 0
- net GND: track 0.00 -> 288.3 mm, vias 0 -> 7
- net VCC: track 284.7 -> 0.00 mm, vias 3 -> 0
- net /SEG0clean: track 0.00 -> 123.5 mm, vias 0 -> 2
- net /SEG2clean: track 0.00 -> 122.7 mm, vias 0 -> 12
- net /SEG1clean: track 0.00 -> 119.7 mm, vias 0 -> 12
- net /SEG3clean: track 0.00 -> 117.3 mm, vias 0 -> 12
- net Net-(BUTTONS1-Pad3): track 113.3 -> 0.00 mm, vias 2 -> 0
- net /COM0clean: track 0.00 -> 111.8 mm, vias 0 -> 2
- net /LOCK: track 0.00 -> 109.8 mm, vias 0 -> 1
- net /SEG4clean: track 0.00 -> 104.8 mm, vias 0 -> 9
- net Net-(BUTTONS1-Pad2): track 101.4 -> 0.00 mm
- net /UNLOCK: track 0.00 -> 92.1 mm, vias 0 -> 2
- net /RESET: track 0.00 -> 91.0 mm, vias 0 -> 1
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- added copper zone on B.Cu, net GND
- added copper zone on F.Cu, net GND
Other:
- board outline added: 100 x 84 mm
- net class Default: clearance 0.2 -> 0.5; trace_width 0.25 -> 0.5
- rule pad_to_mask_clearance: 0 -> 0.2
- rule trace_clearance: 0.2 -> 0.5
- board text added: "ABus CFA100 Display Grabber"
- board text added: "CC-BY 3.0 Sebastian Reichel <sre@mainframe.io>"

Commit message: version 3
Parts:
- added D5: Red LED, LEDs:LED_0805, F.Cu at (171.3, 144.5)
- added R14: 150, Resistors_SMD:R_0805, F.Cu at (171.3, 140.2)
- added U2: PCF8574, Housings_SOIC:SOIC-16_7.5x10.3mm_Pitch1.27mm, F.Cu at (180.3, 142.2)
- P2: value CONN_02X04 -> CONN_01X06; footprint Pin_Headers:Pin_Header_Angled_2x04 -> Pin_Headers:Pin_Header_Angled_1x06
- moved G*** 19.2 mm to (131.1, 132.8)
- moved REF** 16.0 mm to (199.0, 148.0)
- moved REF** 16.0 mm to (109.0, 148.0)
- moved P2 7.55 mm to (177.5, 63.8)
Connections:
- P1 pad 11: /RESET -> /SETUP
- P2 pad 2: /INT -> /SDA
- P2 pad 4: /SDA -> /INT1
- P2 pad 5: /LOCK -> /INT2
- P2 pad 6: /UNLOCK -> GND
- U5 pad 15: (no net) -> /COM0_SEG4
- U7 pad 15: (no net) -> /COM3_SEG4
- U7 pad 18: (no net) -> /COM3_SEG1
- U8 pad 15: (no net) -> /COM4_SEG4
- U9 pad 20: /INT -> /INT1
Routing:
- net /SETUP: track 0.00 -> 150.6 mm, vias 0 -> 1
- net /RESET: track 91.0 -> 0.00 mm, vias 1 -> 0
- net /INT2: track 0.00 -> 84.9 mm, vias 0 -> 1
- net /COM0_SEG4: track 0.00 -> 79.3 mm, vias 0 -> 2
- net /SCL: track 10.7 -> 87.3 mm, vias 0 -> 2
- net /SDA: track 26.4 -> 86.0 mm
- net /COM3_SEG1: track 0.00 -> 48.7 mm, vias 0 -> 2
- net /COM3_SEG4: track 0.00 -> 42.7 mm, vias 0 -> 2
- net /UNLOCK: track 92.1 -> 132.7 mm, vias 2 -> 0
- net GND: track 288.3 -> 318.6 mm
- net /COM4_SEG4: track 0.00 -> 23.9 mm, vias 0 -> 2
- net /INT: track 21.6 -> 0.00 mm, vias 1 -> 0
- net /INT1: track 0.00 -> 20.1 mm, vias 0 -> 1
- net /LED: track 0.00 -> 16.3 mm
- net /LOCK: track 109.8 -> 123.5 mm, vias 1 -> 0
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Other:
- board size 100 x 84 mm -> 100 x 100 mm
- board text added: "ABUS CFA100 Display Grabber"
- board text added: "GND"
- board text added: "INT1"
- board text added: "INT2"
- board text added: "SCL"
- board text added: "SDA"
- board text added: "VCC"
- board text removed: "ABus CFA100 Display Grabber"
