File: acs-display-grabber.sch (KiCad schematic (older format))
At the start: 33 parts, among them IC1 ATMEGA328P-P, U1 74HC14, U2 74HC14

Commit message: version 2
Parts:
- removed BUTTONS1: CONN_01X05, Pin_Headers:Pin_Header_Angled_1x04, symbol CONN_01X04
- removed C1, C2: 22pF, Capacitors_ThroughHole:C_Rect_L7_W2.5_P5, symbol C
- removed C3: 100uF, Capacitors_Elko_ThroughHole:Elko_vert_11.2x6.3mm_RM2.5, symbol C
- removed CRYSTAL1: CRYSTAL, Crystals:Crystal_HC49-U_Vertical, symbol Crystal
- removed D1, D2, D3, D4, D5, D6, D7, D8, D9: ZF 3.9, Diodes_ThroughHole:Diode_DO-35_SOD27_Horizontal_RM10, symbol ZENER
- removed DISPLAY1: CONN_01x09, Pin_Headers:Pin_Header_Angled_1x09, symbol CONN_01X09
- removed I2C_PORT1: CONN_01x04, Pin_Headers:Pin_Header_Angled_1x05, symbol CONN_01X05
- removed IC1: ATMEGA328P-P, Housings_DIP:DIP-28_W7.62mm, symbol ATMEGA328P-P
- removed ISP_PORT1: CONN_02X03, Pin_Headers:Pin_Header_Angled_2x03, symbol CONN_02X03
- removed K?: RELAY_2RT, symbol RELAY_2RT
- removed SUMMER,1: CONN_01X04, Pin_Headers:Pin_Header_Angled_1x04, symbol CONN_01X04
- removed U1, U2: 74HC14, Housings_DIP:DIP-14_W7.62mm, symbol 74HC14
- added C1, C3, C6, C9: 20nF, Capacitors_SMD:C_0805, symbol C_Small
- added C2, C4, C5, C7, C8: 10nF, Capacitors_SMD:C_0805, symbol C_Small
- added D1, D2, D3, D4: 1N4007, Diodes_SMD:MELF_Handsoldering, symbol D
- added P1: CONN_02X07, Pin_Headers:Pin_Header_Angled_2x07, symbol CONN_02X07
- added P2: CONN_02X04, Pin_Headers:Pin_Header_Angled_2x04, symbol CONN_02X04
- added R12, R13: 3.3K, Resistors_SMD:R_0805, symbol R
- added RV1, RV2: POT, ACP CA6:ACP_CA6, symbol POT
- added U1, U4: LM339, Housings_SOIC:SOIC-14_3.9x8.7mm_Pitch1.27mm, symbol LM339
- added U3: LM393, Housings_SOIC:SOIC-8_3.9x4.9mm_Pitch1.27mm, symbol LM393
- added U5, U6, U7, U8: 74LS573, Housings_SOIC:SOIC-20_7.5x12.8mm_Pitch1.27mm, symbol 74LS573
- added U9: MCP23017, Housings_SOIC:SOIC-28_7.5x17.9mm_Pitch1.27mm, symbol MCP23017
- R1, R2, R3, R4: value 470k -> 1.8K; footprint Resistors_ThroughHole:Resistor_Horizontal_RM10mm -> Resistors_SMD:R_0805
- R10, R11, R5, R6, R7, R8, R9: value 470k -> 3.3K; footprint Resistors_ThroughHole:Resistor_Horizontal_RM10mm -> Resistors_SMD:R_0805
Connections:
- net labels added: +5V, COM0, COM0clean, COM1, COM1clean, COM2, COM2clean, COM3, COM3clean, GND, INT, LOCK, RESET, SCL, SDA, SEG0, SEG0clean, SEG1, SEG1clean, SEG2, SEG2clean, SEG3, SEG3clean, SEG4, SEG4clean, UNLOCK, Vhigh, Vlow
- net labels removed: +12V, DISP1, DISP2, DISP3, DISP4, DISP5, DISP6, DISP7, DISP8, DISP9, Earth, I2C_IRQ, ISPRESET, MISO, MOSI, SCK, buzzer, door, reed-switch
- wire segments 174 -> 213
- no-connect marks 3 -> 27

Commit message: version 3
Parts:
- removed P2: CONN_02X04, Pin_Headers:Pin_Header_Angled_2x04, symbol CONN_02X04
- added D5: Red LED, LEDs:LED_0805, symbol LED
- added P2: CONN_01X06, Pin_Headers:Pin_Header_Angled_1x06, symbol CONN_01X06
- added R14: 150, Resistors_SMD:R_0805, symbol R
- added U2: PCF8574, Housings_SOIC:SOIC-16_7.5x10.3mm_Pitch1.27mm, symbol PCF8574
Connections:
- net labels added: COM0_SEG4, COM3_SEG1, COM3_SEG4, COM4_SEG4, INT1, INT2, LED, SETUP
- net labels removed: INT, RESET
- wire segments 213 -> 235
- no-connect marks 27 -> 25
